File: hardware/plug/1v2/Enclosure/0v4_Alu_Sample_76x35/Panel/Front_Panel_76x35.kicad_pcb (KiCad board)
At the start: 2 copper layers, 76 x 35 mm, 11 parts

Commit message: 76x35 sent to fab house
Other:
- outline, holes or cut-outs redrawn
- board text added: "20160819"
- board text added: "8xM2.5 ->"
