File: hardware/plug/1v2/Enclosure/0v4_Alu_Sample_76x35/Panel/Tabs_for_76.kicad_pcb (KiCad board)
At the start: 2 copper layers, 11.5 x 6.9 mm, 1 part, among them P1 CONN_01X01

Commit message: 76x35 sent to fab house
Other:
- board size 11.5 x 6.9 mm -> 11.8 x 6.9 mm
- board text added: "76x35"
- board text added: "LimeSDR"
Changed lines of the file:
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@@
     (links 0)
     (no_connects 0)
-    (area -15.078333 -5.7275 3.360001 9.145001)
+    (area -15.078333 -5.7275 3.360001 9.129958)
     (thickness 1.6)
-    (drawings 1)
+    (drawings 3)
     (tracks 0)
     (zones 0)
@@
     (pad_drill 3.3)
     (pad_to_mask_clearance 0)
-    (aux_axis_origin 0 0)
+    (aux_axis_origin -9.21 -3.68)
     (visible_elements 7FFFFFFF)
     (pcbplotparams
@@
       (viasonmask false)
       (mode 1)
-      (useauxorigin false)
+      (useauxorigin true)
       (hpglpennumber 1)
       (hpglpenspeed 20)
@@
       (psnegative false)
       (psa4output false)
-      (plotreference true)
-      (plotvalue true)
+      (plotreference false)
+      (plotvalue false)
       (plotinvisibletext false)
       (padsonsilk false)
-      (subtractmaskfromsilk false)
+      (subtractmaskfromsilk true)
       (outputformat 1)
       (mirror false)
       (drillshape 0)
       (scaleselection 1)
-      (outputdirectory Gerber/20160710_tabs/))
+      (outputdirectory Gerber/20160819_tabs/))
   )
   (net 0 "")
@@
     (fp_arc (start -2.6 4.349706) (end -3.55 3.058063) (angle 36.33438316) (layer Edge.Cuts) (width 0.02))
     (fp_arc (start -4.698313 -1.553591) (end -4.652118 -3.446725) (angle 35.17359225) (layer Edge.Cuts) (width 0.02))
-    (fp_line (start -8.75 3.447548) (end -4.651552 3.447548) (layer Edge.Cuts) (width 0.02))
-    (fp_line (start -8.75 -3.446725) (end -8.75 3.45) (layer Edge.Cuts) (width 0.02))
-    (fp_line (start -4.652118 -3.446725) (end -8.75 -3.446725) (layer Edge.Cuts) (width 0.02))
+    (fp_line (start -9.1 3.443275) (end -4.651552 3.447548) (layer Edge.Cuts) (width 0.02))
+    (fp_line (start -9.1 -3.446725) (end -9.1 3.443275) (layer Edge.Cuts) (width 0.02))
+    (fp_line (start -4.652118 -3.446725) (end -9.1 -3.446725) (layer Edge.Cuts) (width 0.02))
     (fp_line (start -2.6 2.746322) (end 0 2.746322) (layer Edge.Cuts) (width 0.02))
     (fp_line (start 0 -2.75) (end -2.6 -2.75) (layer Edge.Cuts) (width 0.02))
@@
       (net 1 GND))
   )
-  (dimension 8.75 (width 0.3) (layer Dwgs.User)
-    (gr_text "8.750 mm" (at -4.375 7.75) (layer Dwgs.User)
+  (gr_text LimeSDR (at -5.51 0.02 90) (layer B.SilkS)
+    (effects (font (size 1 1) (thickness 0.1)) (justify mirror))
+  )
+  (gr_text 76x35 (at -5.41 -0.05 90) (layer F.SilkS)
+    (effects (font (size 1 1) (thickness 0.1)))
+  )
+  (dimension 9.100049 (width 0.3) (layer Dwgs.User)
+    (gr_text "9.100 mm" (at -4.575549 7.734957 -0.1888865009) (layer Dwgs.User)
       (effects (font (size 1.5 1.5) (thickness 0.3)))
     )
-    (feature1 (pts (xy -8.75 0) (xy -8.75 9.1)))
-    (feature2 (pts (xy 0 0) (xy 0 9.1)))
-    (crossbar (pts (xy 0 6.4) (xy -8.75 6.4)))
-    (arrow1a (pts (xy -8.75 6.4) (xy -7.623496 5.813579)))
-    (arrow1b (pts (xy -8.75 6.4) (xy -7.623496 6.986421)))
-    (arrow2a (pts (xy 0 6.4) (xy -1.126504 5.813579)))
-    (arrow2b (pts (xy 0 6.4) (xy -1.126504 6.986421)))
+    (feature1 (pts (xy -9.1 -0.03) (xy -9.13 9.06995)))
+    (feature2 (pts (xy 0 0) (xy -0.03 9.09995)))
+    (crossbar (pts (xy -0.021099 6.399965) (xy -9.121099 6.369965)))
+    (arrow1a (pts (xy -9.121099 6.369965) (xy -7.992668 5.787261)))
+    (arrow1b (pts (xy -9.121099 6.369965) (xy -7.996535 6.960096)))
+    (arrow2a (pts (xy -0.021099 6.399965) (xy -1.145663 5.809834)))
+    (arrow2b (pts (xy -0.021099 6.399965) (xy -1.14953 6.982669)))
   )
   (zone (net 0) (net_name "") (layer B.Mask) (hatch edge 0.508)
@@
     (polygon
       (pts
-        (xy -8.87 3.66) (xy -6.71 3.66) (xy -6.73 -3.6) (xy -8.89 -3.6)
+        (xy -9.083005 3.67) (xy -6.923005 3.67) (xy -6.943005 -3.59) (xy -9.103005 -3.59)
       )
     )
@@
     (polygon
       (pts
-        (xy -8.87 3.666033) (xy -6.71 3.666033) (xy -6.73 -3.593967) (xy -8.89 -3.593967)
+        (xy -9.083409 3.666033) (xy -6.923409 3.666033) (xy -6.943409 -3.593967) (xy -9.103409 -3.593967)
       )
     )
@@
     (polygon
       (pts
-        (xy -9.14 -3.76) (xy 3.03 -3.83) (xy 3.36 4.61) (xy -9.37 4.28)
+        (xy -9.39 -3.71) (xy 3.03 -3.83) (xy 3.36 4.61) (xy -9.37 4.28)
       )
     )
@@
     (polygon
       (pts
-        (xy -9.14 -3.767374) (xy 3.03 -3.837374) (xy 3.36 4.602626) (xy -9.37 4.272626)
+        (xy -9.39 -3.73) (xy 3.03 -3.837374) (xy 3.36 4.602626) (xy -9.37 4.272626)
       )
     )
