File: hardware/plug/1v2/Enclosure/0v5_76x35_+4conn/panel/Front_Panel_76x35/Front_Panel_76x35.kicad_pcb (KiCad board)
At the start: 2 copper layers, 76 x 35 mm, 11 parts

Commit message: 3rd batch ready for fab house
Gerber output produced
Combined into a panel

Added small holes on backside for "ventilation" #7
Naming is consistent with current LimeSDR boards W, L, H order for TX #2

Text stays on Silkscreen for now #8
Other:
- board text added: "20160924"
- board text removed: "20160902"
Changed lines of the file:
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@@
-(kicad_pcb (version 4) (host pcbnew "(2016-07-22 BZR 6991, Git 146a78a)-product")
+(kicad_pcb (version 20160815) (host pcbnew "(2016-09-17 revision 679eef1)-makepkg")
   (general
     (links 119)
     (no_connects 0)
-    (area 25.619999 92.929999 101.630001 127.950001)
+    (area 25.34 92.7 101.900001 128.200001)
     (thickness 1.6)
     (drawings 276)
@@
       (drillshape 0)
       (scaleselection 1)
-      (outputdirectory Gerber/20160902_front_panel_10_conn/))
+      (outputdirectory ../_Gerber/20160924_front_panel/))
   )
   (net 0 "")
@@
     (uvia_dia 0.3)
     (uvia_drill 0.1)
+    (diff_pair_gap 0.25)
+    (diff_pair_width 0.2)
     (add_net GND)
   )
@@
   (gr_line (start 26.62 103.06) (end 25.93 103.06) (layer Edge.Cuts) (width 0.02))
   (gr_line (start 26.62 117.9) (end 25.93 117.9) (layer Edge.Cuts) (width 0.02))
-  (gr_text 20160902 (at 95.66 116.33 90) (layer F.Mask)
+  (gr_text 20160924 (at 95.66 116.33 90) (layer F.Mask)
     (effects (font (size 0.8 0.8) (thickness 0.15)) (justify left))
   )
@@
   (gr_line (start 68.8 103.85) (end 68.8 96.03061) (layer B.SilkS) (width 0.5))
   (gr_arc (start 66.74939 103.88) (end 66.69939 105.93) (angle -91.39718103) (layer B.SilkS) (width 0.5))
-  (gr_text L (at 63.05 106.03) (layer B.SilkS)
+  (gr_text W (at 63.05 106.03) (layer B.SilkS)
     (effects (font (size 1.8 1.8) (thickness 0.3)) (justify mirror))
   )
   (gr_line (start 59.25 105.93) (end 53.95 105.93) (layer B.SilkS) (width 0.5))
-  (gr_text W (at 50.05 106.04489) (layer B.SilkS)
+  (gr_text L (at 50.05 106.04489) (layer B.SilkS)
     (effects (font (size 1.8 1.8) (thickness 0.3)) (justify mirror))
   )
@@
     (effects (font (size 1.6 1.6) (thickness 0.3)))
   )
-  (gr_text rx2L (at 62.63 108.01) (layer F.SilkS)
+  (gr_text rx2W (at 62.63 108.01) (layer F.SilkS)
     (effects (font (size 1.6 1.6) (thickness 0.3)))
   )
-  (gr_text rx2W (at 49.91 107.99) (layer F.SilkS)
+  (gr_text rx2L (at 49.91 107.99) (layer F.SilkS)
     (effects (font (size 1.6 1.6) (thickness 0.3)))
   )
@@
     (effects (font (size 1.6 1.6) (thickness 0.3)))
   )
-  (gr_text rx1W (at 49.88 105.57) (layer F.SilkS)
+  (gr_text rx1L (at 49.88 105.57) (layer F.SilkS)
     (effects (font (size 1.6 1.6) (thickness 0.3)))
   )
-  (gr_text rx1L (at 62.58 105.44) (layer F.SilkS)
+  (gr_text rx1W (at 62.58 105.44) (layer F.SilkS)
     (effects (font (size 1.6 1.6) (thickness 0.3)))
   )
@@
     (effects (font (size 1.8 1.8) (thickness 0.3)) (justify mirror))
   )
-  (gr_text W (at 50.05 120.04489) (layer B.SilkS)
+  (gr_text L (at 50.05 120.04489) (layer B.SilkS)
     (effects (font (size 1.8 1.8) (thickness 0.3)) (justify mirror))
   )
-  (gr_text L (at 63.05 120.03) (layer B.SilkS)
+  (gr_text W (at 63.05 120.03) (layer B.SilkS)
     (effects (font (size 1.8 1.8) (thickness 0.3)) (justify mirror))
   )
