File: hardware/plug/1v2/Enclosure/0v6_76x35/panel/Rear_Panel/Rear_Panel_76x35.kicad_pcb (KiCad board)
At the start: 2 copper layers, 76 x 35 mm, 49 parts

Commit message: New Gerbers for 0v6
Parts:
- removed the REF** at (76.4, 118.9)
- removed the REF** at (81.0, 118.9)
- removed the REF** at (76.4, 113.8)
- removed the REF** at (81.0, 113.8)
- added REF**: Hole, Ohisja:hole, F.Cu at (72.8, 98.6)
- added REF**: Hole, Ohisja:hole, F.Cu at (45.4, 98.6)
- added REF**: Hole, Ohisja:hole, F.Cu at (42.4, 98.6)
- added REF**: Hole, Ohisja:hole, F.Cu at (39.3, 98.6)
- added REF**: Hole, Ohisja:hole, F.Cu at (69.8, 98.6)
- added REF**: Hole, Ohisja:hole, F.Cu at (66.7, 98.6)
- added REF**: Hole, Ohisja:hole, F.Cu at (63.7, 98.6)
- added REF**: Hole, Ohisja:hole, F.Cu at (60.6, 98.6)
- added REF**: Hole, Ohisja:hole, F.Cu at (57.6, 98.6)
- added REF**: Hole, Ohisja:hole, F.Cu at (54.5, 98.6)
- added REF**: Hole, Ohisja:hole, F.Cu at (51.5, 98.6)
- added REF**: Hole, Ohisja:hole, F.Cu at (48.4, 98.6)
- added REF1: Hole, Ohisja:hole, F.Cu at (36.3, 98.6)
Other:
- board text added: "20161104"
- board text added: "3.3"
- board text added: "RF Transceiver: Lime Microsystems LMS7002M FPGA: Altera Cyclone IV EP4CE40F23 or EP4CE30F23 Memory: 256 MBytes DDR2 SDRAM Continuous frequency range: 100 kHz – 3.8 GHz Bandwidth: 61.44 MHz Power Output (CW): up to 10 dBm Multiplexing: 2x2 MIMO"
- board text removed: "20161030"
- board text removed: "RF Transceiver: Lime Microsystems LMS7002M MIMO FPRF FPGA: Altera Cyclone IV EP4CE40F23 or EP4CE30F23 Memory: 256 MBytes DDR2 SDRAM Continuous frequency range: 100 kHz – 3.8 GHz Bandwidth: 61.44 MHz Power Output (CW): up to 10 dBm Multiplexing: 2x2 MIMO"
